File: KiCad_Projects/COOLER BASE/COOLER BASE/COOLER BASE.kicad_pcb (KiCad board)
At the start: 2 copper layers, 14.3 x 46.9 mm, 0 parts

Commit message: Added new design
Other:
- board text removed: "PCB3D_BR_"
- board text removed: "PCB3D_TL_"

Commit message: Update files
Other:
- board text added: "SV2IPW"
Changed lines of the file:
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@@
 		(layer "Edge.Cuts")
 	)
+	(gr_text "SV2IPW"
+		(at 117.25 79.26 0)
+		(layer "F.Cu")
+		(effects
+			(font
+				(size 1 1)
+				(thickness 0.15)
+			)
+			(justify left bottom)
+		)
+	)
+	(gr_text "SV2IPW"
+		(at 117.25 79.26 0)
+		(layer "F.Mask")
+		(effects
+			(font
+				(size 1 1)
+				(thickness 0.15)
+			)
+			(justify left bottom)
+		)
+	)
 )
